File: aqm_sensor.kicad_sch (KiCad schematic)
At the start: 12 parts, among them J2 QWIIC, J3 PMS5003, U3 ESP32-C3_SUPERMINI_TH

Commit message: v2 schematic and PCB rework
Schematic:
- Rewire J3 for PMS5003 cable mirror (pin 1↔8 reversal)
- Add I2C pull-up resistors R1, R2 (4.7k) on SDA/SCL
- Replace C4 100uF electrolytic with 10uF 0805 ceramic
- Fix J3 pin types from Unspecified to Passive (ERC clean)
- Add test points: TP1/TP2 (loop) for RX/TX, TP3-TP5 (pad) for power
- Fix C1 value capitalization (0.1uf → 0.1uF)

PCB:
- Rotate U3 180° to correct antenna orientation
- Place new components (R1, R2, C4, TP1-TP5)
- Reroute for updated netlist
- Add GND stitching vias

Removes TODO.md (tracked in CLAUDE.md known issues).

Co-Authored-By: Claude Opus 4.6 (1M context) <noreply@anthropic.com>
Parts:
- added R2, R3: 4.7k, Resistor_SMD:R_1206_3216Metric, symbol Device:R
- added TP1: TX, TestPoint:TestPoint_Loop_D2.50mm_Drill1.0mm, symbol Connector:TestPoint
- added TP2: 3.3V, TestPoint:TestPoint_Pad_D1.5mm, symbol Connector:TestPoint
- added TP3: RX, TestPoint:TestPoint_Loop_D2.50mm_Drill1.0mm, symbol Connector:TestPoint
- added TP4: GND, TestPoint:TestPoint_Pad_D1.5mm, symbol Connector:TestPoint
- added TP5: 5V, TestPoint:TestPoint_Pad_D1.5mm, symbol Connector:TestPoint
- C1: value 0.1uf -> 0.1uF
- C2: renamed from C4; value 100uF -> 10uF; footprint Capacitor_SMD:CP_Elec_5x5.4 -> Capacitor_SMD:C_0805_2012Metric; symbol Device:C_Polarized -> Device:C
- renumbered C2 to C3, H3 to H2, H2 to H3, J3 to J1, R5 to R1, U3 to U1
Connections:
- net +3.3V: now also R2.1, R3.1, TP2.1
- net +5V: now also J1.8, TP5.1; no longer J1.2
- net GND: now also J1.7, TP4.1; no longer J1.1
- net I2C_SCL: now also R2.2
- net I2C_SDA: now also R3.2
- net PMS_RESET: now also J1.3, U1.1 (GPIO1); no longer J1.6, U1.4 (GPIO4)
- net PMS_RX: now also J1.5, U1.3 (GPIO3), TP3.1; no longer J1.4, U1.2 (GPIO2)
- net PMS_SET: now also J1.6, U1.4 (GPIO4); no longer J1.3, U1.1 (GPIO1)
- net PMS_TX: now also U1.2 (GPIO2), TP1.1; no longer U1.3 (GPIO3)
- net at R1.2: now also J1.4; no longer J1.5
- no-connect marks 3 -> 9
Other:
- moved on the sheet: C1, C3, J2, R1

Commit message: Smoke test firmware: WiFi + NTP + MQTT + PMS5003 + HA Discovery
Replaced diagnostic main.c with C++ firmware. Adds WiFi (auto-reconnect,
reduced TX power), NTP, MQTT with LWT, PMS5003 sensor integration, and
HA Discovery for 9 PM/particle entities + RSSI diagnostic. SK6812 LED
reflects PM2.5 levels. Updated CLAUDE.md with architecture analysis and
domain model. Added TODO for ESP-WIFI-MESH migration.

Co-Authored-By: Claude Opus 4.6 (1M context) <noreply@anthropic.com>
Parts:
- H1, H2, H3, H4: value ~ -> (none)
